Commit message: second

File: arduinobot_ws/src/manipulator_description/urdf/arm.urdf.xacro (robot description, xacro)
@@ -1,10 +1,14 @@
 <?xml version="1.0"?>
 <robot xmlns:xacro="http://www.ros.org/wiki/xacro" name="robot_arm">
+    <xacro:property name="PI" value="3.14159"/>
+    <xacro:property name="effort" value="30.0"/>
+    <xacro:property name="velocity" value="10.0"/>
+  <!-- Define world link -->
+  <link name="world"/>
   <!-- Define base link -->
   <link name="base_link">
-    <!-- Define visual representation -->
     <visual>
       <geometry>
-        <cylinder radius="0.5" length="0.5"/>
+        <cylinder radius="0.5" length="0.25"/>
       </geometry>
       <origin xyz="0 0 0" rpy="0 0 0"/>
@@ -13,14 +17,46 @@
       </material>
     </visual>
-    <!-- Define collision representation -->
-    <collision>
+  </link>
+  <!-- Define a joint connecting base_link to the world -->
+  <joint name="virtual_joint" type="fixed">
+    <parent link="world"/>
+    <child link="base_link"/>
+    <origin rpy="0 0 0" xyz="0 0 0"/>
+  </joint>
+  <link name="link_1">
+    <visual>
       <geometry>
-        <cylinder radius="0.25" length="0.5"/>
+        <cylinder radius="0.15" length="1"/>
       </geometry>
-      <origin xyz="0 0 0" rpy="0 0 0"/>
-       <material name="blue">
+      <origin xyz="0 0 0.5" rpy="0 0 0"/>
+      <material name="blue">
         <color rgba="0.1 0.1 0.8 1"/>
       </material>
-    </collision>
+    </visual>
   </link>
+  <joint name="arm_joint" type="revolute">
+    <parent link="base_link"/>
+    <child link="link_1"/>
+    <axis xyz="0 0 1"/>
+    <origin rpy="0 0 0" xyz="0 0 0.125"/>
+    <limit lower="-${PI}" upper="${PI}" effort="${effort}" velocity="${velocity}"/>
+  </joint>
+  <link name="link_2">
+    <visual>
+      <geometry>
+        <cylinder radius="0.15" length="1"/>
+      </geometry>
+      <origin xyz="0 0 0.5" rpy="0 0 0"/>
+      <material name="red">
+        <color rgba="0.8 0.1 0.1 1"/>
+    </material>
+    </visual>
+  </link>
+  <joint name="arm_joint2" type="revolute">
+    <parent link="link_1"/>
+    <child link="link_2"/>
+    <axis xyz="0 1 0"/>
+    <origin rpy="0 0 0" xyz="0 0.3 0.8"/>
+    <limit lower="-${PI}" upper="${PI}" effort="${effort}" velocity="${velocity}"/>
+  </joint>
 </robot>

Commit message: Add files via upload

File: arduinobot_ws/src/manipulator_description/urdf/arm.urdf.xacro (robot description, xacro)
@@ -1,7 +1,4 @@
 <?xml version="1.0"?>
 <robot xmlns:xacro="http://www.ros.org/wiki/xacro" name="robot_arm">
-    <xacro:property name="PI" value="3.14159"/>
-    <xacro:property name="effort" value="30.0"/>
-    <xacro:property name="velocity" value="10.0"/>
   <!-- Define world link -->
   <link name="world"/>
@@ -17,4 +14,13 @@
       </material>
     </visual>
+    <collision>
+      <geometry>
+        <cylinder radius="0.5" length="0.25"/>
+      </geometry>
+    </collision>
+    <inertial>
+      <mass value="1.0"/>
+      <inertia ixx="0.083" ixy="0" ixz="0" iyy="0.083" iyz="0" izz="0.083"/>
+    </inertial>
   </link>
   <!-- Define a joint connecting base_link to the world -->
@@ -24,4 +30,5 @@
     <origin rpy="0 0 0" xyz="0 0 0"/>
   </joint>
+  <!-- Define link_1 with collision and inertia -->
   <link name="link_1">
     <visual>
@@ -34,5 +41,15 @@
       </material>
     </visual>
+    <collision>
+      <geometry>
+        <cylinder radius="0.15" length="1"/>
+      </geometry>
+    </collision>
+    <inertial>
+      <mass value="1.0"/>
+      <inertia ixx="0.025" ixy="0" ixz="0" iyy="0.025" iyz="0" izz="0.025"/>
+    </inertial>
   </link>
+  <!-- Define arm_joint -->
   <joint name="arm_joint" type="revolute">
     <parent link="base_link"/>
@@ -40,6 +57,7 @@
     <axis xyz="0 0 1"/>
     <origin rpy="0 0 0" xyz="0 0 0.125"/>
-    <limit lower="-${PI}" upper="${PI}" effort="${effort}" velocity="${velocity}"/>
+    <limit lower="-3.14159" upper="3.14159" effort="30.0" velocity="10.0"/>
   </joint>
+  <!-- Define link_2 with collision and inertia -->
   <link name="link_2">
     <visual>
@@ -50,7 +68,17 @@
       <material name="red">
         <color rgba="0.8 0.1 0.1 1"/>
-    </material>
+      </material>
     </visual>
+    <collision>
+      <geometry>
+        <cylinder radius="0.15" length="1"/>
+      </geometry>
+    </collision>
+    <inertial>
+      <mass value="1.0"/>
+      <inertia ixx="0.025" ixy="0" ixz="0" iyy="0.025" iyz="0" izz="0.025"/>
+    </inertial>
   </link>
+  <!-- Define arm_joint2 -->
   <joint name="arm_joint2" type="revolute">
     <parent link="link_1"/>
@@ -58,5 +86,5 @@
     <axis xyz="0 1 0"/>
     <origin rpy="0 0 0" xyz="0 0.3 0.8"/>
-    <limit lower="-${PI}" upper="${PI}" effort="${effort}" velocity="${velocity}"/>
+    <limit lower="-3.14159" upper="3.14159" effort="30.0" velocity="10.0"/>
   </joint>
 </robot>
